File: _saved_dc26.sch (KiCad schematic (older format))
At the start: 636 parts

Commit message: Added IR/buttons/etc
Parts:
- CON_IR1: renamed from CON_IR; footprint (none) -> Connectors_JST:JST_PH_B7B-PH-SM4-TB_07x2.00mm_Straight
- gave numbers to parts that had none: 37
- renumbered B_SELECT to B_SELECT1, B_START to B_START1, CON_BTNS to CON_BTNS1, CON_LEDS to CON_LEDS1, CON_PWR to CON_PWR1, IR_RX_F to IR_RX_F1, IR_RX_L to IR_RX_L1, IR_RX_L to IR_RX_L2, IR_RX_R to IR_RX_R1, IR_RX_R to IR_RX_R2, IR_TX_F to IR_TX_F1, PWR_IND to PWR_IND1
