File: dc26-M.kicad_pcb (KiCad board)
At the start: 4 copper layers, 120.1 x 120.1 mm, 638 parts

Commit message: Final coin version
Other:
- board size 120.1 x 120.1 mm -> 120 x 125 mm
Changed lines of the file:
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@@
     (area 115.100046 72.100046 235.399954 192.399954)
     (thickness 1.6)
-    (drawings 1)
+    (drawings 13)
     (tracks 5276)
     (zones 0)
@@
   (layers
     (0 F.Cu signal)
-    (1 GND power hide)
-    (2 VCC power hide)
+    (1 GND power)
+    (2 VCC power)
     (31 B.Cu signal)
     (32 B.Adhes user)
@@
     (pad 1 thru_hole circle (at 0 0) (size 7.5 7.5) (drill 6.2) (layers *.Cu *.Mask F.SilkS))
   )
-  (gr_circle (center 175.25 132.25) (end 235.25 135.25) (layer Edge.Cuts) (width 0.15))
+  (gr_line (start 125 195) (end 135 195) (layer Edge.Cuts) (width 0.15))
+  (gr_line (start 175 190) (end 135 175) (layer Edge.Cuts) (width 0.15))
+  (gr_line (start 125 195) (end 115 195) (layer Edge.Cuts) (width 0.15))
+  (gr_line (start 135 175) (end 135 195) (layer Edge.Cuts) (width 0.15))
+  (gr_line (start 215 175) (end 175 190) (layer Edge.Cuts) (width 0.15))
+  (gr_line (start 215 195) (end 215 175) (layer Edge.Cuts) (width 0.15))
+  (gr_line (start 235 195) (end 215 195) (layer Edge.Cuts) (width 0.15))
+  (gr_line (start 235 70) (end 235 195) (layer Edge.Cuts) (width 0.15))
+  (gr_line (start 215 70) (end 235 70) (layer Edge.Cuts) (width 0.15))
+  (gr_line (start 175 80) (end 215 70) (layer Edge.Cuts) (width 0.15))
+  (gr_line (start 125 70) (end 175 80) (layer Edge.Cuts) (width 0.15))
+  (gr_line (start 115 70) (end 125 70) (layer Edge.Cuts) (width 0.15))
+  (gr_line (start 115 195) (end 115 70) (layer Edge.Cuts) (width 0.15))
   (segment (start 124.9 134.7) (end 125.567762 134.032238) (width 0.25) (layer B.Cu) (net 1))
   (segment (start 123.9 134.7) (end 124.9 134.7) (width 0.25) (layer B.Cu) (net 1))
