File: dc26.sch (KiCad schematic (older format))
At the start: 641 parts, among them U1 STM32F405RGTx

Commit message: moved ICs to top left and connected pins
Parts:
- added J1, J2, J3: CONN_01X10, Pin_Headers:Pin_Header_Angled_1x10_Pitch2.00mm, symbol CONN_01X10
- added U?: TC1262-33VDB, TO_SOT_Packages_SMD:SOT-223, symbol TC1262-33VDB
- R10, R11, R12, R13, R4, R5, R6, R7, R8, R9: value 100R -> 10k
- U2: renamed from U?; footprint (none) -> Housings_DFN_QFN:QFN-24-1EP_4x4mm_Pitch0.5mm
- gave numbers to parts that had none: 3
Connections:
- net +3V3: now also R14.1, U?.3 (VOUT)
- net GND: now also U?.2 (GND), U?.4 (GND)
- net VCC: now also U?.1 (VIN); no longer R14.1
- net at CON_LEDS1.2 (P2), D1.2 (SDI), U1.36 (ADC1_EXTI15/ADC2_EXTI15/ADC3_EXTI15/I2S2_SD/RTC_REFIN/SPI2_MOSI/TIM12_CH2/TIM1_CH3N/TIM8_CH3N/USB_OTG_HS_DP/PB15): now also J3.10 (P10)
- net at CON_LEDS1.1 (P1), D1.3 (CKI), U1.34 (CAN2_TX/I2S2_CK/SPI2_SCK/TIM1_CH1N/USART3_CTS/USB_OTG_HS_ULPI_D6/USB_OTG_HS_VBUS/PB13): now also J3.8 (P8)
- net at U1.10 (PC2/ADC1_IN12/ADC2_IN12/ADC3_IN12/I2S2_ext_SD/SPI2_MISO/USB_OTG_HS_ULPI_DIR): now also J1.8 (P8)
- net at U1.11 (PC3/ADC1_IN13/ADC2_IN13/ADC3_IN13/I2S2_SD/SPI2_MOSI/USB_OTG_HS_ULPI_NXT): now also J1.7 (P7)
- net at U1.2 (PC13/ANTI_TAMP/RTC_AF1): now also J2.7 (P7)
- net at U1.24 (PC4/ADC1_IN14/ADC2_IN14): now also J1.6 (P6)
- net at U1.25 (PC5/ADC1_IN15/ADC2_IN15): now also J1.5 (P5)
- net at U1.29 (I2C2_SCL/I2S2_CK/SPI2_SCK/TIM2_CH3/USART3_TX/USB_OTG_HS_ULPI_D3/PB10): now also J3.5 (P5)
- net at U1.3 (PC14/RCC_OSC32_IN): now also J2.6 (P6)
- net at U1.30 (ADC1_EXTI11/ADC2_EXTI11/ADC3_EXTI11/I2C2_SDA/TIM2_CH4/USART3_RX/USB_OTG_HS_ULPI_D4/PB11): now also J3.6 (P6)
- net at U1.33 (CAN2_RX/I2C2_SMBA/I2S2_WS/SPI2_NSS/TIM1_BKIN/USART3_CK/USB_OTG_HS_ID/USB_OTG_HS_ULPI_D5/PB12): now also J3.7 (P7)
- net at U1.35 (I2S2_ext_SD/SPI2_MISO/TIM12_CH1/TIM1_CH2N/TIM8_CH2N/USART3_RTS/USB_OTG_HS_DM/PB14): now also J3.9 (P9)
- net at U1.37 (PC6/I2S2_MCK/SDIO_D6/TIM3_CH1/TIM8_CH1/USART6_TX): now also J1.4 (P4)
- net at U1.38 (PC7/I2S3_MCK/SDIO_D7/TIM3_CH2/TIM8_CH2/USART6_RX): now also J1.3 (P3)
- net at U1.39 (PC8/SDIO_D0/TIM3_CH3/TIM8_CH3/USART6_CK): now also J1.2 (P2)
- net at U1.4 (PC15/ADC1_EXTI15/ADC2_EXTI15/ADC3_EXTI15/RCC_OSC32_OUT): now also J2.5 (P5)
- net at U1.40 (PC9/DAC_EXTI9/I2C3_SDA/I2S_CKIN/RCC_MCO_2/SDIO_D1/TIM3_CH4/TIM8_CH4): now also J1.1 (P1)
- net at U1.51 (PC10/I2S3_CK/SDIO_D2/SPI3_SCK/UART4_TX/USART3_TX): now also J2.10 (P10)
- net at U1.52 (PC11/ADC1_EXTI11/ADC2_EXTI11/ADC3_EXTI11/I2S3_ext_SD/SDIO_D3/SPI3_MISO/UART4_RX/USART3_RX): now also J2.9 (P9)
- net at U1.53 (PC12/I2S3_SD/SDIO_CK/SPI3_MOSI/UART5_TX/USART3_CK): now also J2.8 (P8)
- net at U1.58 (CAN2_TX/I2C1_SCL/TIM4_CH1/USART1_TX/PB6): now also J3.1 (P1)
- net at U1.59 (I2C1_SDA/TIM4_CH2/USART1_RX/PB7): now also J3.2 (P2)
- net at U1.61 (CAN1_RX/I2C1_SCL/SDIO_D4/TIM10_CH1/TIM4_CH3/PB8): now also J3.3 (P3)
- net at U1.62 (CAN1_TX/DAC_EXTI9/I2C1_SDA/I2S2_WS/SDIO_D5/SPI2_NSS/TIM11_CH1/TIM4_CH4/PB9): now also J3.4 (P4)
- net at U1.8 (PC0/ADC1_IN10/ADC2_IN10/ADC3_IN10/USB_OTG_HS_ULPI_STP): now also J1.10 (P10)
- net at U1.9 (PC1/ADC1_IN11/ADC2_IN11/ADC3_IN11): now also J1.9 (P9)
Other:
- moved on the sheet: PWR_IND1, R14

Commit message: More work on f405
Parts:
- gave numbers to parts that had none: 1

Commit message: F405 schematic almost done
Parts:
- added C? (x2): 2u2, symbol C_Small
- added C? (x5): 0.1pF, symbol C_Small
- added C? (x2): 4u7, symbol CP1
- added C?: 4U7, symbol CP1
- added F405_USB: USB_OTG, symbol USB_OTG
- added JMP-USBID: JMP-USBID, Connectors:GS2, symbol GS2
- added JMP-USBVCC: JMP-USBVCC, Connectors:GS2, symbol GS2
- added PGM: CONN_01X03, symbol CONN_01X03
- added PWR_BATT: LED, LEDs:LED_0603, symbol LED
- added R? (x2): 10k, symbol R_Small
- added R? (x2): 22, symbol R_Small
- added R?: 470R, Resistors_SMD:R_0603, symbol R
- added SW_BOOT0, SW_RESET: SW_SPST, Buttons_Switches_SMD:SW_SPST_EVQQ2, symbol SW_SPST
- added TP-BOOT0: TP-BOOT0, symbol TEST
- added TP-NRST: TP-NRST, symbol TEST
- added TP-PGM-GND: TP-PGM-GND, symbol TEST
- added TP-PGM-SWDCLK: TP-PGM-SWDCLK, symbol TEST
- added TP-PGM-SWDIO: TP-PGM-SWDIO, symbol TEST
- added TP-USBID: TP-USBID, symbol TEST
- R14: value 100R -> 470R
- renumbered PWR_IND1 to PWR_3V3
Connections:
- net +3V3: now also U1.13 (VDDA), C?.1, C?.1, C?.1, C?.2, C?.2, C?.2, R?.1, SW_BOOT0.1 (A)
- net GND: now also U1.12 (VSSA), U1.28 (BOOT1/PB2), C?.1, C?.1, C?.1, C?.2, C?.2, C?.2, C?.2, C?.2, C?.2, C?.2, F405_USB.5 (GND), F405_USB.6 (Shield), PGM.3 (P3), PWR_BATT.2 (A), R?.2, SW_RESET.1 (A), TP-PGM-GND.1
- net VCC: now also C?.1, JMP-USBVCC.1 (G1)
- net at U1.31 (VCAP_1): now also C?.1
- net at U1.42 (DAC_EXTI9/I2C3_SMBA/TIM1_CH2/USART1_TX/USB_OTG_FS_VBUS/PA9): now also C?.1, F405_USB.1 (VBUS), JMP-USBVCC.2 (G2)
- net at U1.43 (TIM1_CH3/USART1_RX/USB_OTG_FS_ID/PA10): now also JMP-USBID.1 (G1)
- net at U1.44 (ADC1_EXTI11/ADC2_EXTI11/ADC3_EXTI11/CAN1_RX/TIM1_CH4/USART1_CTS/USB_OTG_FS_DM/PA11): now also R?.1
- net at U1.45 (CAN1_TX/TIM1_ETR/USART1_RTS/USB_OTG_FS_DP/PA12): now also R?.1
- net at U1.46 (SYS_JTMS-SWDIO/PA13): now also PGM.2 (P2), TP-PGM-SWDIO.1
- net at U1.47 (VCAP_2): now also C?.1
- net at U1.49 (SYS_JTCK-SWCLK/PA14): now also PGM.1 (P1), TP-PGM-SWDCLK.1
- net at U1.60 (BOOT0): now also R?.1, SW_BOOT0.2 (B), TP-BOOT0.1
- net at U1.7 (NRST): now also R?.2, SW_RESET.2 (B), TP-NRST.1
- new net: F405_USB.2 (D-), R?.2
- new net: F405_USB.3 (D+), R?.2
- new net: F405_USB.4 (ID), JMP-USBID.2 (G2), TP-USBID.1
- new net: PWR_BATT.1 (K), R?.2
- new net +BATT: R?.1

Commit message: sub-sheets
Parts:
- removed PWR_BATT: LED, LEDs:LED_0603, symbol LED
- removed R?: 470R, Resistors_SMD:R_0603, symbol R
Connections:
- net BATT-BUCK-ENABLE: now reaches U1.14 (ADC1_IN0/ADC2_IN0/ADC3_IN0/SYS_WKUP/TIM2_CH1/TIM2_ETR/TIM5_CH1/TIM8_ETR/UART4_TX/USART2_CTS/PA0)
Changed lines of the file:
@@
 LIBS:stm32
 LIBS:sensors
+LIBS:dc-dc
 LIBS:dc26-cache
 EELAYER 25 0
@@
 $Descr A4 11693 8268
 encoding utf-8
-Sheet 1 1
+Sheet 1 3
 Title ""
 Date ""
@@
 $EndComp
 $Comp
-L R R?
-U 1 1 5B1A4D77
-P -12350 50
-F 0 "R?" V -12270 50  50  0000 C CNN
-F 1 "470R" V -12350 50  50  0000 C CNN
-F 2 "Resistors_SMD:R_0603" V -12420 50  50  0001 C CNN
-F 3 "" H -12350 50  50  0001 C CNN
-	1    -12350 50
-	0    1    1    0
-$EndComp
-$Comp
-L GND #PWR?
-U 1 1 5B1A4D7D
-P -13150 250
-F 0 "#PWR?" H -13150 0   50  0001 C CNN
-F 1 "GND" H -13150 100 50  0000 C CNN
-F 2 "" H -13150 250 50  0001 C CNN
-F 3 "" H -13150 250 50  0001 C CNN
-	1    -13150 250
-	1    0    0    -1
-$EndComp
-$Comp
-L LED PWR_BATT
-U 1 1 5B1A4D83
-P -12800 50
-F 0 "PWR_BATT" H -12800 150 50  0000 C CNN
-F 1 "LED" H -12800 -50 50  0000 C CNN
-F 2 "LEDs:LED_0603" H -12800 50  50  0001 C CNN
-F 3 "" H -12800 50  50  0001 C CNN
-	1    -12800 50
-	-1   0    0    1
-$EndComp
-$Comp
-L +BATT #PWR?
-U 1 1 5B1AFC40
-P -12100 300
-F 0 "#PWR?" H -12100 150 50  0001 C CNN
-F 1 "+BATT" H -12100 440 50  0000 C CNN
-F 2 "" H -12100 300 50  0001 C CNN
-F 3 "" H -12100 300 50  0001 C CNN
-	1    -12100 300
-	-1   0    0    1
-$EndComp
-$Comp
 L TEST TP-PGM-SWDCLK
 U 1 1 5B1B5199
@@
 	1900 -5400 2700 -5400
 Wire Wire Line
-	2700 -5500 1900 -5500
+	1900 -5500 2700 -5500
 Wire Wire Line
 	1900 -5700 1900 -5900
@@
 Connection ~ -7600 600
 Wire Wire Line
-	-8900 -850 -7950 -850
+	-7950 -850 -8900 -850
 Wire Wire Line
 	-7950 -1400 -7950 1350
@@
 	-9450 3300 -9450 3450
 Wire Wire Line
-	-9850 2900 -10050 2900
+	-10050 2900 -9850 2900
 Wire Wire Line
 	-9050 2900 -8850 2900
@@
 	-11750 4000 -11750 3950
 Wire Wire Line
-	-11300 4750 -11750 4750
+	-11750 4750 -11300 4750
 Wire Wire Line
-	-11750 4750 -11750 4200
+	-11750 4200 -11750 4750
 Wire Wire Line
 	-11850 4350 -11750 4350
@@
 	-12400 4950 -12450 4950
 Wire Wire Line
-	-11300 4950 -12200 4950
+	-12200 4950 -11300 4950
 Wire Wire Line
 	-11850 4750 -11850 4950
@@
 	650  4600 650  4750
 Wire Wire Line
-	-12650 50   -12500 50
-Wire Wire Line
-	-12100 50   -12100 300
-Wire Wire Line
-	-12200 50   -12100 50
-Wire Wire Line
-	-13150 50   -13150 250
-Wire Wire Line
-	-12950 50   -13150 50
-Wire Wire Line
 	-1350 9050 -1350 9200
 Wire Wire Line
@@
 	-7200 2050 -7200 4350
 Wire Wire Line
-	-7100 4350 -7100 2050
+	-7100 2050 -7100 4350
 Wire Wire Line
 	-7200 2050 -6800 2050
@@
 	-6900 8600 -6900 8350
 Connection ~ -7000 8600
+Text GLabel -2000 4750 2    60   Input ~ 0
+BATT-BUCK-ENABLE
+Wire Wire Line
+	-2700 4750 -2000 4750
+$Sheet
+S -21100 -2000 3550 2300
+U 5B2B9E1E
+F0 "batteries" 60
+F1 "batteries.sch" 60
+$EndSheet
+$Sheet
+S -21100 550  3600 2400
+U 5B2CE45B
+F0 "Power Converter" 60
+F1 "power-converter.sch" 60
+$EndSheet
 $EndSCHEMATC

Commit message: mpu6000 circuit complete + power circuit extracted + other changes
Parts:
- removed C? (x2): 4u7, symbol CP1
- removed C?: 4U7, symbol CP1
- removed F405_USB: USB_OTG, symbol USB_OTG
- removed JMP-USBID: JMP-USBID, Connectors:GS2, symbol GS2
- removed JMP-USBVCC: JMP-USBVCC, Connectors:GS2, symbol GS2
- removed PWR_3V3: LED, LEDs:LED_0603, symbol LED
- removed R14: 470R, Resistors_SMD:R_0603, symbol R
- removed R? (x2): 22, symbol R_Small
- removed TP-USBID: TP-USBID, symbol TEST
- removed U2: MPU-6000, Housings_DFN_QFN:QFN-24-1EP_4x4mm_Pitch0.5mm, symbol MPU-6000
- removed U3: TC1262-33VDB, TO_SOT_Packages_SMD:SOT-223, symbol TC1262-33VDB
- gave numbers to parts that had none: 9
- renumbered PGM to PGM1, SW_RESET to SW_RESET1, TP-NRST to TP-NRST1, TP-PGM-GND to TP-PGM-GND1, TP-PGM-SWDCLK to TP-PGM-SWDCLK1, TP-PGM-SWDIO to TP-PGM-SWDIO1
Connections:
- net BATT-BUCK-ENABLE: now also U1.15 (ADC1_IN1/ADC2_IN1/ADC3_IN1/TIM2_CH2/TIM5_CH2/UART4_RX/USART2_RTS/PA1); no longer U1.14 (ADC1_IN0/ADC2_IN0/ADC3_IN0/SYS_WKUP/TIM2_CH1/TIM2_ETR/TIM5_CH1/TIM8_ETR/UART4_TX/USART2_CTS/PA0)
- net MPU6000-INT: now reaches U1.16 (ADC1_IN2/ADC2_IN2/ADC3_IN2/TIM2_CH3/TIM5_CH3/TIM9_CH1/USART2_TX/PA2)
- net MPU6000-CS: now reaches U1.20 (ADC1_IN4/ADC2_IN4/DAC_OUT1/I2S3_WS/SPI1_NSS/SPI3_NSS/USART2_CK/USB_OTG_HS_SOF/PA4)
- net MPU6000-SCLK: now reaches U1.21 (ADC1_IN5/ADC2_IN5/DAC_OUT2/SPI1_SCK/TIM2_CH1/TIM2_ETR/TIM8_CH1N/USB_OTG_HS_ULPI_CK/PA5)
- net MPU6000-MISO: now reaches U1.22 (ADC1_IN6/ADC2_IN6/SPI1_MISO/TIM13_CH1/TIM1_BKIN/TIM3_CH1/TIM8_BKIN/PA6)
- net MPU6000-MOSI: now reaches U1.23 (ADC1_IN7/ADC2_IN7/SPI1_MOSI/TIM14_CH1/TIM1_CH1N/TIM3_CH2/TIM8_CH1N/PA7)
- net USB-VBUS: now reaches U1.42 (DAC_EXTI9/I2C3_SMBA/TIM1_CH2/USART1_TX/USB_OTG_FS_VBUS/PA9)
- net USB-ID: now reaches U1.43 (TIM1_CH3/USART1_RX/USB_OTG_FS_ID/PA10)
- net USB-DM: now reaches U1.44 (ADC1_EXTI11/ADC2_EXTI11/ADC3_EXTI11/CAN1_RX/TIM1_CH4/USART1_CTS/USB_OTG_FS_DM/PA11)
- net USB-DP: now reaches U1.45 (CAN1_TX/TIM1_ETR/USART1_RTS/USB_OTG_FS_DP/PA12)

Commit message: Moved LEDs to new sheet
Parts:
- removed C1, C10, C11, C12, C13, C14, C15, C16, C17, C18, C19, C2, C20, C21, C22, C23, C3, C4, C5, C6, C7, C8, C9: C_Small, Capacitors_SMD:C_0603, symbol C_Small
- removed CON_LEDS1: CONN_01X04, Connectors_JST:JST_GH_BM04B-GHS-TBT_04x1.25mm_Straight, symbol CONN_01X04
- removed D1, D10, D100, D101, D102, D103, D104, D105, D106, D107, D108, D109, D11, D110, D111, D112, D113, D114, D115, D116, D117, D118, D119, D12, D120, D121, D122, D123, D124, D125, D126, D127, D128, D129, D13, D130, D131, D132, D133, D134, D135, D136, D137, D138, D139, D14, D140, D141, D142, D143, D144, D145, D146, D147, D148, D149, D15, D150, D151, D152, D153, D154, D155, D156, D157, D158, D159, D16, D160, D161, D162, D163, D164, D165, D166, D167, D168, D169, D17, D170, D171, D172, D173, D174, D175, D176, D177, D178, D179, D18, D180, D181, D182, D183, D184, D185, D186, D187, D188, D189, D19, D190, D191, D192, D193, D194, D195, D196, D197, D198, D199, D2, D20, D200, D201, D202, D203, D204, D205, D206, D207, D208, D209, D21, D210, D211, D212, D213, D214, D215, D216, D217, D218, D219, D22, D220, D221, D222, D223, D224, D225, D226, D227, D228, D229, D23, D230, D231, D232, D233, D234, D235, D236, D237, D238, D239, D24, D240, D241, D242, D243, D244, D245, D246, D247, D248, D249, D25, D250, D251, D252, D253, D254, D255, D256, D257, D258, D259, D26, D260, D261, D262, D263, D264, D265, D266, D267, D268, D269, D27, D270, D271, D272, D273, D274, D275, D276, D277, D278, D279, D28, D280, D281, D282, D283, D284, D285, D286, D287, D288, D289, D29, D290, D291, D292, D293, D294, D295, D296, D297, D298, D299, D3, D30, D300, D301, D302, D303, D304, D305, D306, D307, D308, D309, D31, D310, D311, D312, D313, D314, D315, D316, D317, D318, D319, D32, D320, D321, D322, D323, D324, D325, D326, D327, D328, D329, D33, D330, D331, D332, D333, D334, D335, D336, D337, D338, D339, D34, D340, D341, D342, D343, D344, D345, D346, D347, D348, D349, D35, D350, D351, D352, D353, D354, D355, D356, D357, D358, D359, D36, D360, D361, D362, D363, D364, D365, D366, D367, D368, D369, D37, D370, D371, D372, D373, D374, D375, D376, D377, D378, D379, D38, D380, D381, D382, D383, D384, D385, D386, D387, D388, D389, D39, D390, D391, D392, D393, D394, D395, D396, D397, D398, D399, D4, D40, D400, D401, D402, D403, D404, D405, D406, D407, D408, D409, D41, D410, D411, D412, D413, D414, D415, D416, D417, D418, D419, D42, D420, D421, D422, D423, D424, D425, D426, D427, D428, D429, D43, D430, D431, D432, D433, D434, D435, D436, D437, D438, D439, D44, D440, D441, D442, D443, D444, D445, D446, D447, D448, D449, D45, D450, D451, D452, D453, D454, D455, D456, D457, D458, D459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: APA102, gsg-modules:APA102-2020, symbol APA102
Connections:
- net LED-SDI: now reaches J3.10 (P10), U1.36 (ADC1_EXTI15/ADC2_EXTI15/ADC3_EXTI15/I2S2_SD/RTC_REFIN/SPI2_MOSI/TIM12_CH2/TIM1_CH3N/TIM8_CH3N/USB_OTG_HS_DP/PB15)
- net LED-CKI: now reaches J3.8 (P8), U1.34 (CAN2_TX/I2S2_CK/SPI2_SCK/TIM1_CH1N/USART3_CTS/USB_OTG_HS_ULPI_D6/USB_OTG_HS_VBUS/PB13)
Other:
- moved on the sheet: CON_PWR1
