File: dc26-challenge/_autosave-dc26-challenge.kicad_pcb (KiCad board)
At the start: 2 copper layers, 107 x 107 mm, 0 parts

Commit message: Final icons + ciphertext
Other:
- board text added: "33, 17, 15, 13, 13, 0d, 43, 0f, 00, 1c, 04, 08, 43, 09, 49, 4c, 07, 0e, 05, 49, 0e, 13, 02, 41, 05, 55, 02, 17, 09, 0d, 04, 1b, 00, 0e, 1a, 0f, 15, 46, 55, 03, 00, 1f, 43, 04, 10, 59, 0a, 06, 01, 06, 14, 41, 00, 0d, 15, 43, 13, 0d, 00, 09, 17, 0d, 14, 14, 45, 50, 11, 1e, 02, 09, 11, 41, 19, 06, 07, 0e, 08, 53"
- board text added: "33, 17, 15, 13, 13, 0d, 47, 08, 13, 1e, 09, 1f, 0c, 50, 11, 04, 06, 47, 12, 52, 1b, 11, 1a, 08, 05, 45, 50, 04, 02, 07, 47, 11, 54, 0f, 16, 17, 41, 09, 46, 50, 0d, 05, 07, 0e, 0c, 47, 5a, 1b, 00, 07, 09, 52, 1d, 04, 18, 0a, 8, 0c"
- board text added: "33, 17, 15, 13, 13, 0d, 53, 0a, 1d, 1c, 08, 02, 49, 05, 08, 40, 43, 06, 42, 50, 08, 1d, 1a, 0e, 1c, 4f, 11, 0b, 4c, 17, 0f, 03, 54, 5a, 11, 0f, 0f, 46, 43, 11, 10, 1f, 06, 47, 05, 41, 09, 06, 1c, 0e, 4b, 49, 1e, 11, 09, 10, 13, 0b, 4e, 1b, 1e, 4e, 08, 0a, 4c, 1e, 00, 1f, 10, 47, 15, 49, 0e, 1a, 4e, 05, 0f, 41, 02, 17, 04, 06, 06, 42, 49, 14, 52, 06, 14, 0b, 41, 1e, 16"
Changed lines of the file:
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@@
     (uvia_drill 0.1)
   )
-  (gr_text "3b, 17, 15, 13, 13, 0d, 0c, 5a, \n21, 1b, 11, 03, 52, 1d, 04, 02, \n44, 14, 42, 50, 1f, 06, 4e, 05, \n09, 47, 50, 0c, 02, 43, 13, 0a, \n45, 5a, 02, 01, 11, 13, 4c, 11, \n17, 4c, 00, 08, 0f, 49, 19, 5e, \n4e, 02, 07, 52, 04, 0a, 03, 0d, \n4b, 42, 41, 14, 16, 4e, 0c, 09, \n56, 19, 00, 4c, 10, 02, 10, 49, \n1f, 01" (at 125.5 121.2) (layer B.SilkS)
+  (gr_text "33, 17, 15, 13, 13, 0d, 53, 0a, \n1d, 1c, 08, 02, 49, 05, 08, 40, \n43, 06, 42, 50, 08, 1d, 1a, 0e, \n1c, 4f, 11, 0b, 4c, 17, 0f, 03, \n54, 5a, 11, 0f, 0f, 46, 43, 11, \n10, 1f, 06, 47, 05, 41, 09, 06, \n1c, 0e, 4b, 49, 1e, 11, 09, 10, \n13, 0b, 4e, 1b, 1e, 4e, 08, 0a, \n4c, 1e, 00, 1f, 10, 47, 15, 49, \n0e, 1a, 4e, 05, 0f, 41, 02, 17, \n04, 06, 06, 42, 49, 14, 52, 06, \n14, 0b, 41, 1e, 16" (at 125 120.6) (layer B.SilkS)
+    (effects (font (size 1.3 1.5) (thickness 0.25)) (justify mirror))
+  )
+  (gr_text "33, 17, 15, 13, 13, 0d, 43, 0f, \n00, 1c, 04, 08, 43, 09, 49, 4c, \n07, 0e, 05, 49, 0e, 13, 02, 41, \n05, 55, 02, 17, 09, 0d, 04, 1b, \n00, 0e, 1a, 0f, 15, 46, 55, 03, \n00, 1f, 43, 04, 10, 59, 0a, 06, \n01, 06, 14, 41, 00, 0d, 15, 43, \n13, 0d, 00, 09, 17, 0d, 14, 14, \n45, 50, 11, 1e, 02, 09, 11, 41, \n19, 06, 07, 0e, 08, 53" (at 74.2 120.4) (layer B.SilkS)
     (effects (font (size 1.5 1.5) (thickness 0.25)) (justify mirror))
   )
-  (gr_text "3b, 17, 15, 13, 13, 0d, 0c, 5a, \n21, 1b, 11, 03, 52, 1d, 04, 02, \n44, 14, 42, 50, 1f, 06, 4e, 05, \n09, 47, 50, 0c, 02, 43, 13, 0a, \n45, 5a, 02, 01, 11, 13, 4c, 11, \n17, 4c, 00, 08, 0f, 49, 19, 5e, \n4e, 02, 07, 52, 04, 0a, 03, 0d, \n4b, 42, 41, 14, 16, 4e, 0c, 09, \n56, 19, 00, 4c, 10, 02, 10, 49, \n1f, 01" (at 74.2 121.3) (layer B.SilkS)
+  (gr_text "33, 17, 15, 13, 13, 0d, 47, 08, \n13, 1e, 09, 1f, 0c, 50, 11, 04, \n06, 47, 12, 52, 1b, 11, 1a, 08, \n05, 45, 50, 04, 02, 07, 47, 11, \n54, 0f, 16, 17, 41, 09, 46, 50, \n0d, 05, 07, 0e, 0c, 47, 5a, 1b, \n00, 07, 09, 52, 1d, 04, 18, 0a, \n8, 0c" (at 125.7 69.9) (layer B.SilkS)
     (effects (font (size 1.5 1.5) (thickness 0.25)) (justify mirror))
   )
-  (gr_text "3b, 17, 15, 13, 13, 0d, 0c, 5a, \n21, 1b, 11, 03, 52, 1d, 04, 02, \n44, 14, 42, 50, 1f, 06, 4e, 05, \n09, 47, 50, 0c, 02, 43, 13, 0a, \n45, 5a, 02, 01, 11, 13, 4c, 11, \n17, 4c, 00, 08, 0f, 49, 19, 5e, \n4e, 02, 07, 52, 04, 0a, 03, 0d, \n4b, 42, 41, 14, 16, 4e, 0c, 09, \n56, 19, 00, 4c, 10, 02, 10, 49, \n1f, 01" (at 125.7 69.9) (layer B.SilkS)
-    (effects (font (size 1.5 1.5) (thickness 0.25)) (justify mirror))
-  )
